File: Control Unit/_restore_backup_2026-06-27T18-06-36-516/Control Unit.kicad_sch (KiCad schematic)
At the start: 17 parts, among them J1 PWR_IN, J2 LM2596S, J3 ST7789, J4 DHT20, J5 RTC, J6 RPM_IN, J7 Page flip, SW1 SW_DPST_x2, U1 ESP32-DEVKIT-V1, U2 PC817

Commit message: rev 1.0
Connections:
- net RPM_PWR_DIODE is gone; now on net RPM_PWR: D2.2 (A), J6.1 (RPM_IN)
- net RPM_PWR_RESISTOR is gone; now on net RPM_PWR: D2.1 (K), R1.1
- net 12V_PWR_BATT: no longer names the net of D1.2 (A), J1.1 (Pin_1)
Changed lines of the file:
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@@
+	(wire
+		(pts
+			(xy 57.15 114.3) (xy 63.5 114.3)
+		)
+		(stroke
+			(width 0)
+			(type default)
+		)
+	)
 	(wire
 		(pts
@@
 		(pts
 			(xy 119.38 85.09) (xy 119.38 82.55)
-		)
-		(stroke
-			(width 0)
-			(type default)
-		)
-	)
-	(wire
-		(pts
-			(xy 57.15 114.3) (xy 63.5 114.3)
 		)
 		(stroke
@@
 		)
 	)
-	(label "RPM_PWR_DIODE"
-		(at 57.15 114.3 0)
+	(label "RPM_PWR"
+		(at 59.69 114.3 0)
 		(effects
 			(font
@@
 		)
 	)
-	(label "12V_PWR_BATT"
-		(at 60.96 80.01 0)
-		(effects
-			(font
-				(size 1.27 1.27)
-			)
-			(justify left bottom)
-		)
-	)
 	(label "3.3V_PWR"
 		(at 151.13 73.66 0)
@@
 		)
 	)
-	(label "RPM_PWR_RESISTOR"
+	(label "RPM_PWR"
 		(at 72.82 114.3 0)
 		(effects
