File: Control Unit/_restore_backup_2026-06-27T18-23-29-983/Control Unit.kicad_pcb (KiCad board)
At the start: 2 copper layers, 100 x 76.5 mm, 17 parts, among them J1 PWR_IN, J2 LM2596S, J3 ST7789, J4 DHT20, J5 RTC, J6 RPM_IN, J7 Page flip, SW1 SW_DPST_x2, U1 ESP32-DEVKIT-V1, U2 PC817

Commit message: rev 1.0
Parts:
- moved U2 25.0 mm to (113.2, 113.7)
- moved D2 16.3 mm to (119.5, 134.5)
Connections:
- net /12V_PWR_BATT renamed Net-(D1-A)
- D2 pad 1: /RPM_PWR_RESISTOR -> /RPM_PWR
- D2 pad 2: /RPM_PWR_DIODE -> /RPM_PWR
- J6 pad 1: /RPM_PWR_DIODE -> /RPM_PWR
- R1 pad 1: /RPM_PWR_RESISTOR -> /RPM_PWR
Routing:
- net Net-(J3-SCL): track 140.4 -> 0.00 mm
- net /3.3V_PWR: track 139.1 -> 0.00 mm
- net Net-(J3-SDA): track 96.0 -> 0.00 mm, vias 4 -> 0
- net Net-(J7-SIG): track 78.6 -> 0.00 mm
- net /12V_PWR: track 43.1 -> 0.00 mm
- net Net-(U1-D34): track 38.7 -> 0.00 mm
- net /3.3V_PWR_SW: track 34.1 -> 0.00 mm
- net Net-(U1-D14): track 31.0 -> 0.00 mm, vias 1 -> 0
- net /RPM_PWR: track 18.8 -> 0.00 mm
- net /RPM_GND: track 16.0 -> 0.00 mm
- net /RPM_PWR_RESISTOR: track 10.8 -> 0.00 mm
- net /RPM_PWR_DIODE: track 9.86 -> 0.00 mm
- net /12V_GND: track 38.8 -> 46.8 mm
- net Net-(D1-A): track 5.46 -> 0.00 mm
- added copper zone on B.Cu, net (none)
- removed copper zone on B.Cu, net GNDREF
Other:
- board size 100 x 76.5 mm -> 100 x 84.5 mm
- board text removed: "Motorcycle Telemetry sensor rev 1.00 Made by: Nguyen Lam Vinh Khang 27/06/2026"
