File: Control Unit/_restore_backup_2026-06-27T18-24-19-349/Control Unit.kicad_pcb (KiCad board)
At the start: 2 copper layers, 100 x 76.5 mm, 17 parts, among them J1 PWR_IN, J2 LM2596S, J3 ST7789, J4 DHT20, J5 RTC, J6 RPM_IN, J7 Page flip, SW1 SW_DPST_x2, U1 ESP32-DEVKIT-V1, U2 PC817

Commit message: rev 1.0
Parts:
- moved U2 15.7 mm to (111.9, 123.0)
Routing:
- net GNDREF: track 0.00 -> 79.1 mm
- net Net-(J3-SCL): track 140.4 -> 96.6 mm
- net Net-(U1-D34): track 38.7 -> 5.09 mm
- net Net-(J3-SDA): track 96.0 -> 64.2 mm, vias 4 -> 3
- net Net-(U1-D14): track 31.0 -> 0.00 mm, vias 1 -> 0
- net /RPM_PWR: track 18.8 -> 0.00 mm
- net /RPM_GND: track 16.0 -> 0.00 mm
- net /12V_PWR: track 43.1 -> 31.0 mm
- net /RPM_PWR_RESISTOR: track 10.8 -> 0.00 mm
- net /RPM_PWR_DIODE: track 9.86 -> 0.00 mm
- net /12V_GND: track 38.8 -> 46.8 mm
- net /3.3V_PWR: track 139.1 -> 144.7 mm
- net Net-(J7-SIG): track 78.6 -> 77.0 mm
- added copper zone on B.Cu, net (none)
- removed copper zone on B.Cu, net GNDREF
Other:
- board text removed: "Motorcycle Telemetry sensor rev 1.00 Made by: Nguyen Lam Vinh Khang 27/06/2026"
